File: sensor-pcb/sensor-pcb.kicad_sch (KiCad schematic)
At the start: 0 parts

Commit message: feat(oled): added oled and button
Parts:
- added SW1: SW_Push_Dual, Button_Switch_THT:SW_SPST_Omron_B3F-40xx, symbol Switch:SW_Push_Dual
- added U1: ESP32-C6-DevKitC-1, PCM_Espressif:ESP32-C6-DevKitC-1, symbol PCM_Espressif:ESP32-C6-DevKitC-1
- added U2: ~, Connector_PinSocket_2.54mm:PinSocket_1x08_P2.54mm_Vertical, symbol my_lib:ens160_aht20_board
- added U3: ~, Connector_PinSocket_2.54mm:PinSocket_1x06_P2.54mm_Horizontal, symbol my_lib:sd_card_board
- added U4: ~, Connector_PinSocket_2.54mm:PinSocket_1x04_P2.54mm_Vertical, symbol my_lib:i2c_oled
Connections:
- new net +3.3V: U1.1 (3V3), U2.2 (3V3), U4.2 (VCC)
- new net +5V: U1.14 (5V), U2.1 (VIN), U3.2 (VCC)
- new net CS: U1.25 (GPIO20), U3.6 (CS)
- new net GND: SW1.1, SW1.3, U1.15 (GND), U1.18 (GND), U1.21 (GND), U1.32 (GND), U2.3 (GND), U3.1 (GND), U4.1 (GND)
- new net GPIO5: SW1.2, SW1.4, U1.4 (GPIO5/MTDI)
- new net MISO: U1.26 (GPIO21), U3.3 (MISO)
- new net MOSI: U1.27 (GPIO22), U3.4 (MOSI)
- new net SCK: U1.24 (GPIO19), U3.5 (SCK)
- new net SCL: U1.6 (GPIO7), U2.4 (SCL), U4.3 (SCL)
- new net SDA: U1.5 (GPIO6), U2.5 (SDA), U4.4 (SDA)
- no-connect marks 0 -> 3
